Commit message: real robot a little bit rotated relative a table

File: willbot_description/urdf/willbot.urdf.xacro (robot description, xacro)
@@ -14,5 +14,5 @@
       <parent link="world"/>
       <child link = "base_link"/>
-      <origin xyz="0.0 0.0 0.0" rpy="0.0 0.0 0.0"/>
+      <origin xyz="0.0 0.0 0.0" rpy="0.0 0.01 0.0"/>
     </joint>
   </xacro:if>
