Commit message: add force-torque sensor to the paris urdf model. Change xacro namespace

File: willbot_description/urdf/adapter.grenoble.macro.xacro (robot description, xacro)
@@ -4,5 +4,5 @@
 Adapter between arm and gripper for Paris setup.
 -->
-<robot xmlns:xacro="http://ros.org/wiki/xacro">
+<robot xmlns:xacro="http://wiki.ros.org/xacro">
   <xacro:macro name="grenoble_adapter" params="prefix">
     <xacro:property name="adapter_radius" value="0.040" />

File: willbot_description/urdf/adapter.paris.macro.xacro (robot description, xacro)
@@ -4,6 +4,6 @@
 Adapter between arm and gripper for Grenoble setup.
 -->
-<robot xmlns:xacro="http://ros.org/wiki/xacro">
-  <xacro:macro name="paris_adapter" params="prefix">
+<robot xmlns:xacro="http://wiki.ros.org/xacro">
+  <xacro:macro name="paris_adapter" params="prefix parent *origin">
     <xacro:property name="adapter_radius" value="0.040" />
     <xacro:property name="adapter_length" value="0.030" />
@@ -13,6 +13,6 @@
     <xacro:property name="tube_remove" value="0.100" />
     <joint name="${prefix}tool0-adapter_fixed_joint" type="fixed">
-      <origin xyz="0 0 0" rpy="0 0 ${-pi/4}"/>
-      <parent link="${prefix}tool0"/>
+      <xacro:insert_block name="origin"/>
+      <parent link="${parent}"/>
       <child link="${prefix}adapter_link"/>
     </joint>

File: willbot_description/urdf/willbot.macro.xacro (robot description, xacro)
@@ -6,14 +6,16 @@
 there are multiple arms then a prefix followed by an "_" is needed.
 -->
-<robot xmlns:xacro="http://ros.org/wiki/xacro">
-  <!-- robotiq s model -->
-  <xacro:include filename="$(find robotiq_3f_gripper_visualization)/cfg/robotiq-3f-gripper_articulated_macro.xacro" />
+<robot xmlns:xacro="http://wiki.ros.org/xacro">
   <!-- common stuff -->
   <xacro:include filename="$(find ur_description)/urdf/common.gazebo.xacro" />
   <!-- ur5 -->
   <xacro:include filename="$(find ur_description)/urdf/ur5.urdf.xacro" />
+  <!-- force torque sensor -->
+  <xacro:include filename="$(find willbot_description)/urdf/robotiq_fts.macro.xacro" />
   <!-- adapter -->
   <xacro:include filename="$(find willbot_description)/urdf/adapter.paris.macro.xacro" />
   <xacro:include filename="$(find willbot_description)/urdf/adapter.grenoble.macro.xacro" />
+  <!-- robotiq s model -->
+  <xacro:include filename="$(find robotiq_3f_gripper_visualization)/cfg/robotiq-3f-gripper_articulated_macro.xacro" />
   <xacro:macro name="willbot" params="prefix setup">
     <!-- arm -->
@@ -37,9 +39,22 @@
         wrist_3_lower_limit="${-pi}" wrist_3_upper_limit="${pi}" />
     </xacro:if>
+    <!-- Connect tool0_controller to base using floating joint -->
+    <!-- This frame will be sending by the UR5 driver with take into account the arm calibration -->
+    <joint name="base_tool0_controller_floating_joint" type="floating">
+      <origin xyz="0 0 0" rpy="0 0 0"/>
+      <parent link="base"/>
+      <child link="tool0_controller"/>
+    </joint>
+    <link name="tool0_controller"/>
     <!-- hand -->
     <xacro:robotiq-3f-gripper_articulated prefix="${prefix}hand_"/>
     <!-- arm to hand adapter -->
     <xacro:if value="${setup == 'paris'}">
-      <xacro:paris_adapter prefix="${prefix}"/>
+      <xacro:robotiq_fts prefix="${prefix}" parent="${prefix}tool0">
+        <origin rpy="0 0 0" xyz="0 0 0.002"/>
+      </xacro:robotiq_fts>
+      <xacro:paris_adapter prefix="${prefix}" parent="${prefix}fts_toolside">
+        <origin rpy="0 0 ${pi+pi/12}" xyz="0 0 0"/>
+      </xacro:paris_adapter>
     </xacro:if>
     <xacro:if value="${setup == 'grenoble'}">

File: willbot_description/urdf/willbot.urdf.xacro (robot description, xacro)
@@ -1,4 +1,4 @@
 <?xml version="1.0"?>
-<robot xmlns:xacro="http://ros.org/wiki/xacro" name="willbot">
+<robot xmlns:xacro="http://wiki.ros.org/xacro" name="willbot">
   <xacro:include filename="$(find willbot_description)/urdf/willbot.macro.xacro" />
   <xacro:arg name="setup" default=""/>
