Commit message: formatting

File: willbot_description/urdf/willbot.macro.xacro (robot description, xacro)
@@ -14,73 +14,56 @@
   <xacro:include filename="$(find ur_description)/urdf/ur5.urdf.xacro" />
   <xacro:macro name="willbot" params="prefix">
-  	  <!-- arm -->
-  	  <!-- be careful, shoulder_pan has limits -2pi..0 -->
-  	  <xacro:ur5_robot prefix="${prefix}" joint_limited="true"
-    	shoulder_pan_lower_limit="${-2*pi}" shoulder_pan_upper_limit="${0}"
-    	shoulder_lift_lower_limit="${-pi}" shoulder_lift_upper_limit="${pi}"
-    	elbow_joint_lower_limit="${-pi}" elbow_joint_upper_limit="${pi}"
-    	wrist_1_lower_limit="${-pi}" wrist_1_upper_limit="${pi}"
-    	wrist_2_lower_limit="${-pi}" wrist_2_upper_limit="${pi}"
-    	wrist_3_lower_limit="${-pi}" wrist_3_upper_limit="${pi}"
-  	  />
-  	  <!-- hand -->
-	  <xacro:s-model_articulated prefix="${prefix}hand_"/>
-	  <!-- arm to hand adapter -->
-	  <xacro:property name="adapter_radius" value="0.040" />
-	  <xacro:property name="adapter_length" value="0.025" />
-	  <xacro:property name="adapter_weight" value="0.100" />
-	  <joint name="${prefix}tool0-adapter_fixed_joint" type="fixed">
-        <origin xyz="0 0 0" rpy="0 0 0"/>
-        <parent link="${prefix}tool0"/>
-        <child link="${prefix}adapter_link"/>
-      </joint>
-	  <link name="${prefix}adapter_link">
-        <visual>
-          <origin xyz="0.0 0.0 ${adapter_length/2.0}" rpy="0 0 0" />
-          <geometry>
-            <cylinder radius="${adapter_radius}" length="${adapter_length}"/>
-          </geometry>
-          <material name="Grey">
-            <color rgba="0.2 0.2 0.2 1.0"/>
-          </material>
-        </visual>
-        <collision>
-          <origin xyz="0.0 0.0 ${adapter_length/2.0}" rpy="0 0 0" />
-          <geometry>
-            <cylinder radius="${adapter_radius}" length="${adapter_length}"/>
-          </geometry>
-        </collision>
-        <xacro:cylinder_inertial radius="${adapter_radius}" length="${adapter_length}" mass="${adapter_weight}">
-          <origin xyz="0.0 0.0 ${adapter_length/2.0}" rpy="0 0 0" />
-        </xacro:cylinder_inertial>
-      </link>
-      <joint name="${prefix}adapter-palm_fixed_joint" type="fixed">
-        <origin xyz="0 0 ${adapter_length+0.045}" rpy="${pi/2} 0 ${-pi/4}"/>
-        <parent link="${prefix}adapter_link"/>
-        <child link="${prefix}hand_palm"/>
-      </joint>
-      <!-- tool position -->
-      <link name="${prefix}tool" />
-      <joint name="${prefix}adapter_link-tool_joint" type="fixed">
-        <origin  rpy="0 0 ${-pi/4}" xyz="0 0 ${adapter_length+0.2}"/>
-        <parent link="${prefix}tool0"/>
-        <child link="${prefix}tool"/>
-      </joint>
-	  <!-- objects -->
- 	  <!--link name="table_link">
-        <visual>
-          <geometry>
-            <box size="1 1 0.1" />
-          </geometry>
-          <material name="LightGrey">
-            <color rgba="0.7 0.7 0.7 1.0"/>
-          </material>
-        </visual>
-        <collision>
-          <geometry>
-            <box size="1 1 0.1" />
-          </geometry>
-        </collision>
-      </link-->
+    <!-- arm -->
+    <!-- be careful, shoulder_pan has limits -2pi..0 -->
+    <xacro:ur5_robot prefix="${prefix}" joint_limited="true"
+      shoulder_pan_lower_limit="${-2*pi}" shoulder_pan_upper_limit="${0}"
+      shoulder_lift_lower_limit="${-pi}" shoulder_lift_upper_limit="${pi}"
+      elbow_joint_lower_limit="${-pi}" elbow_joint_upper_limit="${pi}"
+      wrist_1_lower_limit="${-pi}" wrist_1_upper_limit="${pi}"
+      wrist_2_lower_limit="${-pi}" wrist_2_upper_limit="${pi}"
+      wrist_3_lower_limit="${-pi}" wrist_3_upper_limit="${pi}" />
+    <!-- hand -->
+    <xacro:s-model_articulated prefix="${prefix}hand_"/>
+    <!-- arm to hand adapter -->
+    <xacro:property name="adapter_radius" value="0.040" />
+    <xacro:property name="adapter_length" value="0.025" />
+    <xacro:property name="adapter_weight" value="0.100" />
+    <joint name="${prefix}tool0-adapter_fixed_joint" type="fixed">
+      <origin xyz="0 0 0" rpy="0 0 0"/>
+      <parent link="${prefix}tool0"/>
+      <child link="${prefix}adapter_link"/>
+    </joint>
+    <link name="${prefix}adapter_link">
+      <visual>
+        <origin xyz="0.0 0.0 ${adapter_length/2.0}" rpy="0 0 0" />
+        <geometry>
+          <cylinder radius="${adapter_radius}" length="${adapter_length}"/>
+        </geometry>
+        <material name="Grey">
+          <color rgba="0.2 0.2 0.2 1.0"/>
+        </material>
+      </visual>
+      <collision>
+        <origin xyz="0.0 0.0 ${adapter_length/2.0}" rpy="0 0 0" />
+        <geometry>
+          <cylinder radius="${adapter_radius}" length="${adapter_length}"/>
+        </geometry>
+      </collision>
+      <xacro:cylinder_inertial radius="${adapter_radius}" length="${adapter_length}" mass="${adapter_weight}">
+        <origin xyz="0.0 0.0 ${adapter_length/2.0}" rpy="0 0 0" />
+      </xacro:cylinder_inertial>
+    </link>
+    <joint name="${prefix}adapter-palm_fixed_joint" type="fixed">
+      <origin xyz="0 0 ${adapter_length+0.045}" rpy="${pi/2} 0 ${-pi/4}"/>
+      <parent link="${prefix}adapter_link"/>
+      <child link="${prefix}hand_palm"/>
+    </joint>
+    <!-- tool position -->
+    <link name="${prefix}tool" />
+    <joint name="${prefix}adapter_link-tool_joint" type="fixed">
+      <origin rpy="0 0 ${-pi/4}" xyz="0 0 ${adapter_length+0.2}"/>
+      <parent link="${prefix}tool0"/>
+      <child link="${prefix}tool"/>
+    </joint>
   </xacro:macro>
 </robot>

Commit message: change model

File: willbot_description/urdf/willbot.macro.xacro (robot description, xacro)
@@ -13,9 +13,9 @@
   <!-- ur5 -->
   <xacro:include filename="$(find ur_description)/urdf/ur5.urdf.xacro" />
-  <xacro:macro name="willbot" params="prefix">
+  <xacro:macro name="willbot" params="prefix shoulder_pan_zero:=${-pi} adapter_length:=${0.025} adapter_rotation:=${0.0}">
     <!-- arm -->
     <!-- be careful, shoulder_pan has limits -2pi..0 -->
     <xacro:ur5_robot prefix="${prefix}" joint_limited="true"
-      shoulder_pan_lower_limit="${-2*pi}" shoulder_pan_upper_limit="${0}"
+      shoulder_pan_lower_limit="${shoulder_pan_zero-pi}" shoulder_pan_upper_limit="${shoulder_pan_zero+pi}"
       shoulder_lift_lower_limit="${-pi}" shoulder_lift_upper_limit="${pi}"
       elbow_joint_lower_limit="${-pi}" elbow_joint_upper_limit="${pi}"
@@ -27,5 +27,5 @@
     <!-- arm to hand adapter -->
     <xacro:property name="adapter_radius" value="0.040" />
-    <xacro:property name="adapter_length" value="0.025" />
+    <!--xacro:property name="adapter_length" value="0.025" /-->
     <xacro:property name="adapter_weight" value="0.100" />
     <joint name="${prefix}tool0-adapter_fixed_joint" type="fixed">
@@ -55,5 +55,5 @@
     </link>
     <joint name="${prefix}adapter-palm_fixed_joint" type="fixed">
-      <origin xyz="0 0 ${adapter_length+0.045}" rpy="${pi/2} 0 ${-pi/4}"/>
+      <origin xyz="0 0 ${adapter_length+0.045}" rpy="${pi/2} 0 ${adapter_rotation-pi/4}"/>
       <parent link="${prefix}adapter_link"/>
       <child link="${prefix}hand_palm"/>

File: willbot_description/urdf/willbot.urdf.xacro (robot description, xacro)
@@ -2,10 +2,10 @@
 <robot xmlns:xacro="http://ros.org/wiki/xacro" name="willbot">
   <xacro:include filename="$(find willbot_description)/urdf/willbot.macro.xacro" />
-  <xacro:willbot prefix=""/>
+  <xacro:willbot prefix="" shoulder_pan_zero="${-pi/2}" adapter_length="${0.084}" adapter_rotation="${pi}"/>
   <link name="world" />
   <joint name="world_joint" type="fixed">
 	<parent link="world" />
 	<child link = "base_link" />
-	<origin xyz="0.0 0.0 0.0" rpy="0.0 0.0 0.0" />
+	<origin xyz="0.0 0.0 0.0" rpy="0.0 0.0 ${-pi/2}" />
   </joint>
 </robot>

Commit message: switch to a kinetic branch of a robotiq stack

File: willbot_description/urdf/willbot.macro.xacro (robot description, xacro)
@@ -8,5 +8,5 @@
 <robot xmlns:xacro="http://ros.org/wiki/xacro">
   <!-- robotiq s model -->
-  <xacro:include filename="$(find robotiq_s_model_visualization)/cfg/s-model_articulated_macro.xacro" />
+  <xacro:include filename="$(find robotiq_3f_gripper_visualization)/cfg/robotiq-3f-gripper_articulated_macro.xacro" />
   <!-- common stuff -->
   <xacro:include filename="$(find ur_description)/urdf/common.gazebo.xacro" />
@@ -24,5 +24,5 @@
       wrist_3_lower_limit="${-pi}" wrist_3_upper_limit="${pi}" />
     <!-- hand -->
-    <xacro:s-model_articulated prefix="${prefix}hand_"/>
+    <xacro:robotiq-3f-gripper_articulated prefix="${prefix}hand_"/>
     <!-- arm to hand adapter -->
     <xacro:property name="adapter_radius" value="0.040" />

File: willbot_description/urdf/willbot.urdf (robot description, URDF)
Before this commit: robot willbot, 27 links, 26 joints
Links:
- link hand_finger_1_link_0: geometry collision mesh filename=package://robotiq_3f_gripper_visualization/meshes/s-model_a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; visual mesh filename=package://robotiq_3f_gripper_visualization/meshes/s-model_a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
- link hand_finger_1_link_1: geometry collision mesh filename=package://robotiq_3f_gripper_visualization/meshes/s-model_a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; visual mesh filename=package://robotiq_3f_gripper_visualization/meshes/s-model_a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
- link hand_finger_1_link_2: geometry collision mesh filename=package://robotiq_3f_gripper_visualization/meshes/s-model_a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; visual mesh filename=package://robotiq_3f_gripper_visualization/meshes/s-model_a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
- link hand_finger_1_link_3: geometry collision mesh filename=package://robotiq_3f_gripper_visualization/meshes/s-model_a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; visual mesh filename=package://robotiq_3f_gripper_visualization/meshes/s-model_a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
- link hand_finger_2_link_0: geometry collision mesh filename=package://robotiq_3f_gripper_visualization/meshes/s-model_a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; visual mesh filename=package://robotiq_3f_gripper_visualization/meshes/s-model_a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
- link hand_finger_2_link_1: geometry collision mesh filename=package://robotiq_3f_gripper_visualization/meshes/s-model_a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; visual mesh filename=package://robotiq_3f_gripper_visualization/meshes/s-model_a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
- link hand_finger_2_link_2: geometry collision mesh filename=package://robotiq_3f_gripper_visualization/meshes/s-model_a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; visual mesh filename=package://robotiq_3f_gripper_visualization/meshes/s-model_a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
- link hand_finger_2_link_3: geometry collision mesh filename=package://robotiq_3f_gripper_visualization/meshes/s-model_a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; visual mesh filename=package://robotiq_3f_gripper_visualization/meshes/s-model_a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
- link hand_finger_middle_link_0: geometry collision mesh filename=package://robotiq_3f_gripper_visualization/meshes/s-model_a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; visual mesh filename=package://robotiq_3f_gripper_visualization/meshes/s-model_a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
- link hand_finger_middle_link_1: geometry collision mesh filename=package://robotiq_3f_gripper_visualization/meshes/s-model_a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; visual mesh filename=package://robotiq_3f_gripper_visualization/meshes/s-model_a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
- link hand_finger_middle_link_2: geometry collision mesh filename=package://robotiq_3f_gripper_visualization/meshes/s-model_a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; visual mesh filename=package://robotiq_3f_gripper_visualization/meshes/s-model_a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
- link hand_finger_middle_link_3: geometry collision mesh filename=package://robotiq_3f_gripper_visualization/meshes/s-model_a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; visual mesh filename=package://robotiq_3f_gripper_visualization/meshes/s-model_a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
- link hand_palm: geometry collision mesh filename=package://robotiq_3f_gripper_visualization/meshes/s-model_a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; visual mesh filename=package://robotiq_3f_gripper_visualization/meshes/s-model_a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

Commit message: add collision for cable protection

File: willbot_description/urdf/willbot.macro.xacro (robot description, xacro)
@@ -30,5 +30,5 @@
     <xacro:property name="adapter_weight" value="0.100" />
     <joint name="${prefix}tool0-adapter_fixed_joint" type="fixed">
-      <origin xyz="0 0 0" rpy="0 0 0"/>
+      <origin xyz="0 0 0" rpy="0 0 ${-pi/4}"/>
       <parent link="${prefix}tool0"/>
       <child link="${prefix}adapter_link"/>
@@ -50,4 +50,10 @@
         </geometry>
       </collision>
+      <collision>
+        <origin xyz="0.055 0.0 0.035" rpy="0 0 0" />
+        <geometry>
+          <box size="0.11 0.09 0.07" />
+        </geometry>
+      </collision>
       <xacro:cylinder_inertial radius="${adapter_radius}" length="${adapter_length}" mass="${adapter_weight}">
         <origin xyz="0.0 0.0 ${adapter_length/2.0}" rpy="0 0 0" />
@@ -55,5 +61,5 @@
     </link>
     <joint name="${prefix}adapter-palm_fixed_joint" type="fixed">
-      <origin xyz="0 0 ${adapter_length+0.045}" rpy="${pi/2} 0 ${-pi/4}"/>
+      <origin xyz="0 0 ${adapter_length+0.045}" rpy="${pi/2} 0 0"/>
       <parent link="${prefix}adapter_link"/>
       <child link="${prefix}hand_palm"/>
@@ -66,4 +72,11 @@
       <child link="${prefix}tool"/>
     </joint>
+    <!-- hand palm plane position -->
+    <link name="${prefix}hand_palm_plane" />
+    <joint name="${prefix}adapter_link-hand_palm_plane" type="fixed">
+      <origin rpy="0 0 ${-pi/4}" xyz="0 0 ${adapter_length+0.095}"/>
+      <parent link="${prefix}tool0"/>
+      <child link="${prefix}hand_palm_plane"/>
+    </joint>
   </xacro:macro>
 </robot>

Commit message: common robot description for paris and grenoble

File: willbot_description/urdf/willbot.macro.xacro (robot description, xacro)
@@ -13,68 +13,49 @@
   <!-- ur5 -->
   <xacro:include filename="$(find ur_description)/urdf/ur5.urdf.xacro" />
-  <xacro:macro name="willbot" params="prefix">
+  <!-- adapter -->
+  <xacro:include filename="$(find willbot_description)/urdf/adapter.paris.macro.xacro" />
+  <xacro:include filename="$(find willbot_description)/urdf/adapter.grenoble.macro.xacro" />
+  <xacro:macro name="willbot" params="prefix setup">
     <!-- arm -->
-    <!-- be careful, shoulder_pan has limits -2pi..0 -->
-    <xacro:ur5_robot prefix="${prefix}" joint_limited="true"
-      shoulder_pan_lower_limit="${-2*pi}" shoulder_pan_upper_limit="${0}"
-      shoulder_lift_lower_limit="${-pi}" shoulder_lift_upper_limit="${pi}"
-      elbow_joint_lower_limit="${-2*pi}" elbow_joint_upper_limit="${0}"
-      wrist_1_lower_limit="${-2*pi}" wrist_1_upper_limit="${0}"
-      wrist_2_lower_limit="${-pi}" wrist_2_upper_limit="${pi}"
-      wrist_3_lower_limit="${-pi}" wrist_3_upper_limit="${pi}" />
+    <!-- be careful with non-stardart joint limits -->
+    <xacro:if value="${setup == 'paris'}">
+      <xacro:ur5_robot prefix="${prefix}" joint_limited="true"
+        shoulder_pan_lower_limit="${-2*pi}" shoulder_pan_upper_limit="${0}"
+        shoulder_lift_lower_limit="${-pi}" shoulder_lift_upper_limit="${pi}"
+        elbow_joint_lower_limit="${-2*pi}" elbow_joint_upper_limit="${0}"
+        wrist_1_lower_limit="${-2*pi}" wrist_1_upper_limit="${0}"
+        wrist_2_lower_limit="${-pi}" wrist_2_upper_limit="${pi}"
+        wrist_3_lower_limit="${-pi}" wrist_3_upper_limit="${pi}" />
+    </xacro:if>
+    <xacro:if value="${setup == 'grenoble'}">
+      <xacro:ur5_robot prefix="${prefix}" joint_limited="true"
+        shoulder_pan_lower_limit="${-3*pi/2}" shoulder_pan_upper_limit="${pi/2}"
+        shoulder_lift_lower_limit="${-pi}" shoulder_lift_upper_limit="${pi}"
+        elbow_joint_lower_limit="${-2*pi}" elbow_joint_upper_limit="${0}"
+        wrist_1_lower_limit="${-pi}" wrist_1_upper_limit="${pi}"
+        wrist_2_lower_limit="${-pi}" wrist_2_upper_limit="${pi}"
+        wrist_3_lower_limit="${-pi}" wrist_3_upper_limit="${pi}" />
+    </xacro:if>
     <!-- hand -->
     <xacro:robotiq-3f-gripper_articulated prefix="${prefix}hand_"/>
     <!-- arm to hand adapter -->
-    <xacro:property name="adapter_radius" value="0.040" />
-    <xacro:property name="adapter_length" value="0.025" />
-    <xacro:property name="adapter_weight" value="0.100" />
-    <joint name="${prefix}tool0-adapter_fixed_joint" type="fixed">
-      <origin xyz="0 0 0" rpy="0 0 ${-pi/4}"/>
-      <parent link="${prefix}tool0"/>
-      <child link="${prefix}adapter_link"/>
-    </joint>
-    <link name="${prefix}adapter_link">
-      <visual>
-        <origin xyz="0.0 0.0 ${adapter_length/2.0}" rpy="0 0 0" />
-        <geometry>
-          <cylinder radius="${adapter_radius}" length="${adapter_length}"/>
-        </geometry>
-        <material name="Grey">
-          <color rgba="0.2 0.2 0.2 1.0"/>
-        </material>
-      </visual>
-      <collision>
-        <origin xyz="0.0 0.0 ${adapter_length/2.0}" rpy="0 0 0" />
-        <geometry>
-          <cylinder radius="${adapter_radius}" length="${adapter_length}"/>
-        </geometry>
-      </collision>
-      <collision>
-        <origin xyz="0.055 0.0 0.035" rpy="0 0 0" />
-        <geometry>
-          <box size="0.11 0.09 0.07" />
-        </geometry>
-      </collision>
-      <xacro:cylinder_inertial radius="${adapter_radius}" length="${adapter_length}" mass="${adapter_weight}">
-        <origin xyz="0.0 0.0 ${adapter_length/2.0}" rpy="0 0 0" />
-      </xacro:cylinder_inertial>
-    </link>
-    <joint name="${prefix}adapter-palm_fixed_joint" type="fixed">
-      <origin xyz="0 0 ${adapter_length+0.045}" rpy="${pi/2} 0 0"/>
-      <parent link="${prefix}adapter_link"/>
-      <child link="${prefix}hand_palm"/>
-    </joint>
+    <xacro:if value="${setup == 'paris'}">
+      <xacro:paris_adapter prefix="${prefix}"/>
+    </xacro:if>
+    <xacro:if value="${setup == 'grenoble'}">
+      <xacro:grenoble_adapter prefix="${prefix}"/>
+    </xacro:if>
     <!-- tool position -->
     <link name="${prefix}tool" />
-    <joint name="${prefix}adapter_link-tool_joint" type="fixed">
-      <origin rpy="0 0 ${-pi/4}" xyz="0 0 ${adapter_length+0.2}"/>
-      <parent link="${prefix}tool0"/>
+    <joint name="${prefix}hand_base-tool_joint" type="fixed">
+      <origin rpy="0 0 0" xyz="0 0 0.2"/>
+      <parent link="${prefix}hand_base"/>
       <child link="${prefix}tool"/>
     </joint>
     <!-- hand palm plane position -->
     <link name="${prefix}hand_palm_plane" />
-    <joint name="${prefix}adapter_link-hand_palm_plane" type="fixed">
-      <origin rpy="0 0 ${-pi/4}" xyz="0 0 ${adapter_length+0.095}"/>
-      <parent link="${prefix}tool0"/>
+    <joint name="${prefix}hand_base-hand_palm_plane" type="fixed">
+      <origin rpy="0 0 0" xyz="0 0 0.05"/>
+      <parent link="${prefix}hand_base"/>
       <child link="${prefix}hand_palm_plane"/>
     </joint>

File: willbot_description/urdf/willbot.urdf.xacro (robot description, xacro)
@@ -2,10 +2,25 @@
 <robot xmlns:xacro="http://ros.org/wiki/xacro" name="willbot">
   <xacro:include filename="$(find willbot_description)/urdf/willbot.macro.xacro" />
-  <xacro:willbot prefix=""/>
-  <link name="world" />
-  <joint name="world_joint" type="fixed">
-	<parent link="world" />
-	<child link = "base_link" />
-	<origin xyz="0.0 0.0 0.0" rpy="0.0 0.0 0.0" />
-  </joint>
+  <xacro:arg name="setup" default=""/>
+  <xacro:arg name="prefix" default=""/>
+  <xacro:property name="setup" value="$(arg setup)"/>
+  <xacro:property name="prefix" value="$(arg prefix)"/>
+  <!-- robot -->
+  <xacro:willbot setup="${setup}" prefix="${prefix}"/>
+  <!-- connect to the world link -->
+  <link name="world"/>
+  <xacro:if value="${setup == 'paris'}">
+    <joint name="world_joint" type="fixed">
+      <parent link="world"/>
+      <child link = "base_link"/>
+      <origin xyz="0.0 0.0 0.0" rpy="0.0 0.0 0.0"/>
+    </joint>
+  </xacro:if>
+  <xacro:if value="${setup == 'grenoble'}">
+    <joint name="world_joint" type="fixed">
+      <parent link="world"/>
+      <child link = "base_link"/>
+      <origin xyz="0.0 0.0 0.0" rpy="0.0 0.0 ${-pi/2}"/>
+    </joint>
+  </xacro:if>
 </robot>

Commit message: update description to the new paris configuration

File: willbot_description/urdf/willbot.macro.xacro (robot description, xacro)
@@ -23,5 +23,5 @@
     <xacro:if value="${setup == 'paris'}">
       <xacro:ur5_robot prefix="${prefix}" joint_limited="true"
-        shoulder_pan_lower_limit="${-2*pi}" shoulder_pan_upper_limit="${0}"
+        shoulder_pan_lower_limit="${-pi}" shoulder_pan_upper_limit="${pi}"
         shoulder_lift_lower_limit="${-pi}" shoulder_lift_upper_limit="${pi}"
         elbow_joint_lower_limit="${-2*pi}" elbow_joint_upper_limit="${0}"
@@ -32,5 +32,5 @@
     <xacro:if value="${setup == 'grenoble'}">
       <xacro:ur5_robot prefix="${prefix}" joint_limited="true"
-        shoulder_pan_lower_limit="${-3*pi/2}" shoulder_pan_upper_limit="${pi/2}"
+        shoulder_pan_lower_limit="${-pi}" shoulder_pan_upper_limit="${pi}"
         shoulder_lift_lower_limit="${-pi}" shoulder_lift_upper_limit="${pi}"
         elbow_joint_lower_limit="${-2*pi}" elbow_joint_upper_limit="${0}"

File: willbot_description/urdf/willbot.urdf.xacro (robot description, xacro)
@@ -14,5 +14,5 @@
       <parent link="world"/>
       <child link = "base_link"/>
-      <origin xyz="0.0 0.0 0.0" rpy="0.0 0.01 0.0"/>
+      <origin xyz="0.0 0.0 0.003" rpy="0.0 0.0 ${-pi/2}"/>
     </joint>
   </xacro:if>
