Commit message: add tube collision geometry to paris setup

File: willbot_description/urdf/adapter.paris.macro.xacro (robot description, xacro)
@@ -9,4 +9,7 @@
     <xacro:property name="adapter_length" value="0.025" />
     <xacro:property name="adapter_weight" value="0.100" />
+    <xacro:property name="tube_length" value="0.100" />
+    <xacro:property name="tube_radius" value="0.022" />
+    <xacro:property name="tube_remove" value="0.100" />
     <joint name="${prefix}tool0-adapter_fixed_joint" type="fixed">
       <origin xyz="0 0 0" rpy="0 0 ${-pi/4}"/>
@@ -36,4 +39,10 @@
         </geometry>
       </collision>
+      <collision>
+        <origin xyz="${tube_remove} 0.0 ${-tube_length/2.0 + 0.02}" rpy="0 0 0" />
+        <geometry>
+          <cylinder radius="${tube_radius}" length="${tube_length}"/>
+        </geometry>
+      </collision>
       <xacro:cylinder_inertial radius="${adapter_radius}" length="${adapter_length}" mass="${adapter_weight}">
         <origin xyz="0.0 0.0 ${adapter_length/2.0}" rpy="0 0 0" />

Commit message: add new adapter part between the robot and the gripper into the URDF model

File: willbot_description/urdf/adapter.paris.macro.xacro (robot description, xacro)
@@ -7,5 +7,5 @@
   <xacro:macro name="paris_adapter" params="prefix">
     <xacro:property name="adapter_radius" value="0.040" />
-    <xacro:property name="adapter_length" value="0.025" />
+    <xacro:property name="adapter_length" value="0.030" />
     <xacro:property name="adapter_weight" value="0.100" />
     <xacro:property name="tube_length" value="0.100" />

Commit message: add stuff for HTC vive trackers

File: willbot_description/urdf/adapter.paris.macro.xacro (robot description, xacro)
@@ -62,4 +62,17 @@
       <child link="${prefix}hand_palm"/>
     </joint>
+    <!-- vive tracker mount -->
+    <link name="${prefix}tool_mount"/>
+    <link name="${prefix}tool_tracker"/>
+    <joint name="${prefix}tool0-tool_mount-fixed_joint" type="fixed">
+      <origin xyz="0 0 0" rpy="0 0 ${-pi*5/12}"/> <!-- 115-180 grad -->
+      <parent link="${prefix}tool0"/>
+      <child link="${prefix}tool_mount"/>
+    </joint>
+    <joint name="${prefix}tool_mount-tool_tracker-fixed_joint" type="fixed">
+      <origin xyz="0 -0.120 0.004" rpy="0 0 0"/>
+      <parent link="${prefix}tool_mount"/>
+      <child link="${prefix}tool_tracker"/>
+    </joint>
   </xacro:macro>
 </robot>

Commit message: correct arm collision model for paris setup

File: willbot_description/urdf/adapter.paris.macro.xacro (robot description, xacro)
@@ -11,5 +11,5 @@
     <xacro:property name="tube_length" value="0.100" />
     <xacro:property name="tube_radius" value="0.022" />
-    <xacro:property name="tube_remove" value="0.100" />
+    <xacro:property name="tube_remove" value="0.080" />
     <joint name="${prefix}tool0-adapter_fixed_joint" type="fixed">
       <xacro:insert_block name="origin"/>
@@ -34,7 +34,13 @@
       </collision>
       <collision>
-        <origin xyz="0.055 0.0 0.035" rpy="0 0 0" />
+        <origin xyz="0.06 -0.025 0.06" rpy="0 1.57 0" />
         <geometry>
-          <box size="0.11 0.09 0.07" />
+          <cylinder radius="0.01" length="0.05"/>
+        </geometry>
+      </collision>
+      <collision>
+        <origin xyz="0.06 0.025 0.06" rpy="0 1.57 0" />
+        <geometry>
+          <cylinder radius="0.01" length="0.05"/>
         </geometry>
       </collision>

Commit message: change collision model for Paris setup

File: willbot_description/urdf/adapter.paris.macro.xacro (robot description, xacro)
@@ -9,5 +9,5 @@
     <xacro:property name="adapter_length" value="0.030" />
     <xacro:property name="adapter_weight" value="0.100" />
-    <xacro:property name="tube_length" value="0.100" />
+    <xacro:property name="tube_length" value="0.160" />
     <xacro:property name="tube_radius" value="0.022" />
     <xacro:property name="tube_remove" value="0.080" />
@@ -46,5 +46,5 @@
       </collision>
       <collision>
-        <origin xyz="${tube_remove} 0.0 ${-tube_length/2.0 + 0.02}" rpy="0 0 0" />
+        <origin xyz="${tube_remove} 0.0 ${-tube_length/2.0}" rpy="0 0 0" />
         <geometry>
           <cylinder radius="${tube_radius}" length="${tube_length}"/>
